Commit message: added continuous joints to wheels, robot can now move forward at constant speed

File: Sim_code/URDF/diff_drive.urdf (robot description, URDF)
Before this commit: robot test_robot, 6 links, 5 joints
Joints:
- joint base_to_lwheel: axis (none) -> 0 0 1; limit (none) -> effort=1 velocity=1000; origin xyz=0 0.115 0.046 rpy=1.5708 0 0 -> xyz=-0.05 0.115 0.046 rpy=-1.5708 0 0; type fixed -> continuous
- joint base_to_rwheel: axis (none) -> 0 0 1; limit (none) -> effort=1 velocity=1000; origin xyz=0 -0.115 0.046 rpy=-1.5708 0 0 -> xyz=-0.05 -0.115 0.046 rpy=-1.5708 0 0; type fixed -> continuous

Commit message: added score tracker for ball contact, tested backward movement, but backward doesn't straight in a line like forward does

File: Sim_code/URDF/diff_drive.urdf (robot description, URDF)
Before this commit: robot test_robot, 6 links, 5 joints
Links:
- link base_link: mass 3.0 -> 6.0
- link caster_wheel: mass 0.1 -> 5
- link lwheel: mass 0.5 -> 3
- link rwheel: mass 0.5 -> 3
- link scanner: mass 0.05 -> 5

Commit message: changed wheel geometry and fc, implemented a forward function and camera module lock on the scanner of the robot. However, robot still slides a little after it reach target distance

File: Sim_code/URDF/diff_drive.urdf (robot description, URDF)
Before this commit: robot test_robot, 6 links, 5 joints
Links:
- link caster_mount: mass 0.001 -> 5
- link lwheel: geometry collision mesh filename=stl/pololu-wheel-80x10mm-black.stl scale=0.001 0.001 0.001; visual mesh filename=stl/pololu-wheel-80x10mm-black.stl scale=0.001 0.001 0.001
- link rwheel: geometry collision mesh filename=stl/pololu-wheel-80x10mm-black.stl scale=0.001 0.001 0.001; visual mesh filename=stl/pololu-wheel-80x10mm-black.stl scale=0.001 0.001 0.001

Commit message: fixing world coordinate orientation, map scan has fixed coordinates and adding printHeading function printing current robot heading based don compass setting.

File: Sim_code/URDF/diff_drive.urdf (robot description, URDF)
Before this commit: robot test_robot, 6 links, 5 joints
Links:
- link caster_wheel: mass 5 -> 10
